File: pcb/ampselector.kicad_pcb (KiCad board)
At the start: 2 copper layers, 85 x 100 mm, 24 parts, among them SW1 SW_Push, SW10 RotaryEncoder_Switch, SW2 SW_Push, SW3 SW_Push, SW4 SW_Push, SW5 SW_Push, SW6 SW_Push, SW7 SW_Push, SW8 SW_Push, SW9 RotaryEncoder_Switch, U1 MOUDLE-SEEEDUINO-XIAO, U2 ER_OLEDM0.91_1x-I2C

Commit message: updates to PCB and case and general design
Parts:
- moved U1 14.1 mm to (57.0, 83.5), turned to -90 degrees
Routing:
- net Net-(U1-PA11_A3_D3): track 104.7 -> 211.6 mm
- net GND: track 98.5 -> 165.1 mm
- net Net-(U1-PA6_A10_D10_MOSI): track 69.6 -> 105.4 mm
- net Net-(U1-PA5_A9_D9_MISO): track 41.3 -> 74.2 mm
- net Net-(U1-PA02_A0_D0): track 43.8 -> 76.5 mm, vias 0 -> 1
- net Net-(U1-PA10_A2_D2): track 72.0 -> 96.3 mm
- net Net-(D1-K): track 199.6 -> 220.1 mm, vias 0 -> 1
- net Net-(U1-PB09_A7_D7_RX): track 17.1 -> 36.8 mm
- net VCC: track 28.9 -> 47.4 mm, vias 0 -> 2
- net Net-(U1-PA4_A1_D1): track 95.5 -> 112.9 mm
- net Net-(U1-PA7_A8_D8_SCK): track 50.0 -> 63.8 mm
- net Net-(D10-K): track 140.6 -> 131.4 mm
- net Net-(U1-PB08_A6_D6_TX): track 34.4 -> 43.1 mm
Other:
- board text added: "RAVINDER DADIALA @ravinder-Olivier v1.0.0 AMPSELECTOR"
- board text removed: "RAVINDER OLIVIER SINGH DADIALA @ravinder-Olivier v1.0.0 AMPSELECTOR"
